File: KiCad/Electronic Speed Controller/ESC Files/ESC/BLOCK DIAGRAM.kicad_sch (KiCad schematic)
At the start: 0 parts

Commit message: Create ESC block diagram
Other:
- note added: "0-60V"
- note added: "CAN"
- note added: "COM"
- note added: "ESC BLOCK DIAGRAM"
- note added: "HALL/ENCODER"
- note added: "MCU"
- note added: "MOSFET_DRIVER"
- note added: "MOSFETs"
- note added: "MOTOR"
- note added: "SERVO"
- note added: "TEMP_SENSOR"
- note added: "USB"
- note added: "V_SUPPLY"
- company: (none) -> Alpha Amps
- title: (none) -> ESC Block Diagram
