File: KiCad/Electronic Speed Controller/ESC/BLOCK DIAGRAM.kicad_sch (KiCad schematic)
At the start: 0 parts

Commit message: Update MCU schematic file
Other:
- note added: "${TITLE}"
- note removed: "ESC BLOCK DIAGRAM"
Changed lines of the file:
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@@
 		)
 	)
-	(text "ESC BLOCK DIAGRAM"
+	(text "${TITLE}"
 		(exclude_from_sim no)
 		(at 153.162 23.114 0)
